File: ccat-board.kicad_pcb (KiCad board)
At the start: 2 copper layers, 43 parts, among them J1 JTAG, J2 UART, J3 USB_B_Micro, Q1 Q_NPN_BCE, Q2 Q_NPN_BEC, SW1 SW_Push, SW2 SW_Push, U1 ESP32-C3-MINI-1-N4, U2 CP2102N-A02-GQFN28, U3 AMS1117-3.3

Commit message: Add files.
Parts:
- added J4: Conn_01x15_Female, Connector_PinHeader_2.54mm:PinHeader_1x15_P2.54mm_Vertical, F.Cu at (55.6, 74.8)
- added J5: Conn_01x15_Female, Connector_PinHeader_2.54mm:PinHeader_1x15_P2.54mm_Vertical, F.Cu at (89.5, 74.5)
- C4: value 22pf -> 22pF
- D5: value RED LED -> LED
- R15: value 5K1 -> 1k5
Connections:
- D2 pad 1: /D- -> IO18
- D3 pad 1: /D+ -> IO19
- J3 pad 2: /D- -> IO18
- J3 pad 3: /D+ -> IO19
