File: ccat-board.kicad_sch (KiCad schematic)
At the start: 45 parts, among them J1 JTAG, J2 UART, J3 USB_B_Micro, J4 Conn_01x15, J5 Conn_01x15, Q1 Q_NPN_BCE, Q2 Q_NPN_BEC, SW1 SW_Push, SW2 SW_Push, U1 ESP32-C3-MINI-1-N4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

Commit message: Add files.
Parts:
- removed C8: 1uF, Capacitor_SMD:C_0402_1005Metric, symbol Device:C
- removed C9: 10uF, Capacitor_SMD:C_0603_1608Metric, symbol Device:C
- removed J4, J5: Conn_01x15, symbol Connector_Generic:Conn_01x15
- removed R10: 22K1, Resistor_SMD:R_0402_1005Metric, symbol Device:R
- removed R11: 1K, Resistor_SMD:R_0402_1005Metric, symbol Device:R
- removed R12, R13, R3, R4, R5, R6: 0, Resistor_SMD:R_0402_1005Metric, symbol Device:R
- removed R14: 10K, Resistor_SMD:R_0402_1005Metric, symbol Device:R
- removed R9: 47K5, Resistor_SMD:R_0402_1005Metric, symbol Device:R
- removed U2: CP2102N-A02-GQFN28, Package_DFN_QFN:QFN-28-1EP_5x5mm_P0.5mm_EP3.35x3.35mm, symbol Interface_USB:CP2102N-Axx-xQFN28
- added J4, J5: Conn_01x15_Female, Connector_PinHeader_2.54mm:PinHeader_1x15_P2.54mm_Vertical, symbol Connector:Conn_01x15_Female
- C4: value 22pf -> 22pF
- D5: value RED LED -> LED
- R15: value 5K1 -> 1k5
Connections:
- net D+ is gone; now on net IO19: D3.1 (A1), J3.3 (D+)
- net D- is gone; now on net IO18: D2.1 (A1), J3.2 (D-)
- net +3.3V: now also J4.2 (Pin_2), J4.3 (Pin_3)
- net +5V: now also J4.13 (Pin_13), J4.14 (Pin_14)
- net EN: now also J4.7 (Pin_7)
- net GND: now also J4.1 (Pin_1), J4.12 (Pin_12), J4.15 (Pin_15), J4.6 (Pin_6), J4.8 (Pin_8), J5.1 (Pin_1), J5.12 (Pin_12), J5.15 (Pin_15), J5.4 (Pin_4), J5.7 (Pin_7)
- net IO0: now also J4.9 (Pin_9)
- net IO1: now also J4.10 (Pin_10)
- net IO10: now also J4.11 (Pin_11)
- net IO18: now also J5.13 (Pin_13)
- net IO19: now also J5.14 (Pin_14)
- net IO2: now also J4.4 (Pin_4)
- net IO3: now also J4.5 (Pin_5)
- net IO4: now also J5.11 (Pin_11)
- net IO5: now also J5.10 (Pin_10)
- net IO6: now also J5.9 (Pin_9)
- net IO7: now also J5.8 (Pin_8)
- net IO8: now also J5.6 (Pin_6)
- net IO9: now also J5.5 (Pin_5)
- net U0RXD: now also J5.3 (Pin_3)
- net U0TXD: now also J5.2 (Pin_2)
- no-connect marks 17 -> 2
Other:
- moved on the sheet: D5, Q1, Q2, R15, R16, R17
